Commit message: Update firefly.xacro

File: rotors_description/urdf/firefly.xacro (robot description, xacro)
@@ -10,5 +10,5 @@
   You may obtain a copy of the License at
   http://www.apache.org/licenses/LICENSE-2.0
-  Unless required by applicable law or agreed to in writing, software
+  Unless requiDarkGrey by applicable law or agreed to in writing, software
   distributed under the License is distributed on an "AS IS" BASIS,
   WITHOUT WARRANTIES OR CONDITIONS OF ANY KIND, either express or implied.
@@ -22,5 +22,5 @@
   <xacro:property name="use_mesh_file" value="true" />
   <xacro:property name="mesh_file" value="package://rotors_description/meshes/firefly.dae" />
-  <xacro:property name="mass" value="1.5" /> <!-- [kg] -->
+  <xacro:property name="mass" value="1.5" /> <!-- [kg] --><!--original one is 1.5-->
   <xacro:property name="body_width" value="0.1" /> <!-- [m] -->
   <xacro:property name="body_height" value="0.16" /> <!-- [m] -->
@@ -48,4 +48,5 @@
   <!-- Included URDF Files -->
   <xacro:include filename="$(find rotors_description)/urdf/multirotor_base.xacro" />
+  <!--<xacro:include filename="$(find subt_gazebo)/urdf/led.urdf.xacro" />-->
   <!-- Instantiate multirotor_base_macro once -->
   <xacro:multirotor_base_macro
@@ -56,4 +57,5 @@
     use_mesh_file="${use_mesh_file}"
     mesh_file="${mesh_file}"
+    color ="DarkGrey"
     >
     <xacro:insert_block name="body_inertia" />
@@ -75,5 +77,5 @@
     rotor_drag_coefficient="${rotor_drag_coefficient}"
     rolling_moment_coefficient="${rolling_moment_coefficient}"
-    color="Red"
+    color="DarkGrey"
     use_own_mesh="false"
     mesh="">
@@ -96,5 +98,5 @@
     rotor_drag_coefficient="${rotor_drag_coefficient}"
     rolling_moment_coefficient="${rolling_moment_coefficient}"
-    color="Blue"
+    color="DarkGrey"
     use_own_mesh="false"
     mesh="">
@@ -116,5 +118,5 @@
     rotor_drag_coefficient="${rotor_drag_coefficient}"
     rolling_moment_coefficient="${rolling_moment_coefficient}"
-    color="Blue"
+    color="DarkGrey"
     use_own_mesh="false"
     mesh="">
@@ -136,5 +138,5 @@
     rotor_drag_coefficient="${rotor_drag_coefficient}"
     rolling_moment_coefficient="${rolling_moment_coefficient}"
-    color="Blue"
+    color="DarkGrey"
     use_own_mesh="false"
     mesh="">
@@ -157,5 +159,5 @@
     rotor_drag_coefficient="${rotor_drag_coefficient}"
     rolling_moment_coefficient="${rolling_moment_coefficient}"
-    color="Blue"
+    color="DarkGrey"
     use_own_mesh="false"
     mesh="">
@@ -178,5 +180,5 @@
     rotor_drag_coefficient="${rotor_drag_coefficient}"
     rolling_moment_coefficient="${rolling_moment_coefficient}"
-    color="Red"
+    color="DarkGrey"
     use_own_mesh="false"
     mesh="">
@@ -184,3 +186,24 @@
     <xacro:insert_block name="rotor_inertia" />
   </xacro:vertical_rotor>
+<!--Instantiate the led-->
+ <!-- <xacro:led led_prefix="main" parent_link="${namespace}/base_link">
+    <pose>0 0 0.3 0 0 0</pose>
+    <params>
+      <block>
+         <duration>0.3</duration>
+         <interval>0.3</interval>
+         <color>1 0 0</color>
+      <block>
+      <block>
+         <duration>0.3</duration>
+         <interval>0.3</interval>
+         <color>0 1 0</color>
+      <block>
+      <block>
+         <duration>0.3</duration>
+         <interval>0.3</interval>
+         <color>0 0 1</color>
+      <block>
+    </params>
+  </xacro:led>-->
 </robot>
